Commit message: Changelog
-) New caster wheel model
-) Removed actuation of caster wheels
-) Slipping and bouncing bug fixes

File: wheelchair_description/urdf/wheelchair_body.xacro (robot description, xacro)
@@ -1,4 +1,11 @@
 <?xml version="1.0"?>
 <robot xmlns:xacro="http://www.ros.org/wiki/xacro">
+	<!-- Base Footprint -->
+	<link name="base_footprint"/>
+	<joint name="base_footprint_joint" type="fixed">
+		<origin xyz="0 0 ${wheel_radius + 0.125}" rpy="0 0 0" /> <!-- 0.125 distanza centro ruota>base_link -->
+		<parent link="base_footprint"/>
+		<child link="base_link" />
+	</joint>
 	<!-- Base Link -->
 	<link name="base_link">
@@ -14,5 +21,13 @@
 		<inertial>
 			<mass value="${base_mass}"/>
-			<inertia ixx="0.13" ixy="0.0" ixz="0.0" iyx="0.0" iyy="0.21" iyz="0.0" izx="0.0" izy="0.0" izz="0.13"/>
+			<inertia ixx="${base_mass*inertia_correcting_factor*(base_z*base_z+base_x*base_x)/12}"
+					 ixy="0.0"
+					 ixz="0.0"
+					 iyx="0.0"
+					 iyy="${base_mass*inertia_correcting_factor*(base_y*base_y+base_x*base_x)/12}"
+					 iyz="0.0"
+					 izx="0.0"
+					 izy="0.0"
+					 izz="${base_mass*inertia_correcting_factor*(base_y*base_y+base_z*base_z)/12}"/>
 		</inertial>
 	</link>

File: wheelchair_description/urdf/wheelchair_gazebo.xacro (robot description, xacro)
@@ -39,23 +39,56 @@
   	</gazebo>
 	<!-- Ruote -->
-	<gazebo reference="$left_wheel">
-		<material>Gazebo/Grey</material>
-	</gazebo>
-	<gazebo reference="$right_wheel">
-		<material>Gazebo/Grey</material>
+	<gazebo reference="left_wheel">
+		<material>Gazebo/Grey</material>
+		<kp>1000000.0</kp>
+		<kd>10.0</kd>
+		<mu1>1.5</mu1>
+		<mu2>1.5</mu2>
+		<fdir1>1 0 0</fdir1>
+		<maxVel>1.0</maxVel>
+		<minDepth>0.00</minDepth>
+	</gazebo>
+	<gazebo reference="right_wheel">
+		<material>Gazebo/Grey</material>
+		<kp>1000000.0</kp>
+		<kd>1.0</kd>
+		<mu1>1</mu1>
+		<mu2>1</mu2>
+		<fdir1>1 0 0</fdir1>
+		<maxVel>1.0</maxVel>
+		<minDepth>0.00</minDepth>
 	</gazebo>
 	<!-- Caster -->
-	<gazebo reference="left_caster">
-		<material>Gazebo/Grey</material>
-	</gazebo>
-	<gazebo reference="right_caster">
-		<material>Gazebo/Grey</material>
-	</gazebo>
-	<!-- Top -->
-	<gazebo reference="left_top">
-		<material>Gazebo/White</material>
-	</gazebo>
-	<gazebo reference="right_top">
-		<material>Gazebo/White</material>
+	<gazebo reference="left_castor_wheel_link">
+		<material>Gazebo/Grey</material>
+		<kp>1000000.0</kp>
+		<kd>1.0</kd>
+		<mu1>0.25</mu1>
+		<mu2>0.25</mu2>
+		<fdir1>1 0 0</fdir1>
+		<maxVel>1.0</maxVel>
+		<minDepth>0.00</minDepth>
+	</gazebo>
+	<gazebo reference="right_castor_wheel_link">
+		<material>Gazebo/Grey</material>
+		<kp>1000000.0</kp>
+		<kd>1.0</kd>
+		<mu1>0.25</mu1>
+		<mu2>0.25</mu2>
+		<fdir1>1 0 0</fdir1>
+		<maxVel>1.0</maxVel>
+		<minDepth>0.00</minDepth>
+	</gazebo>
+	<gazebo reference="left_castor_mount_link">
+		<material>Gazebo/DarkGrey</material>
+	</gazebo>
+	<gazebo reference="right_castor_mount_link">
+		<material>Gazebo/DarkGrey</material>
+	</gazebo>
+	<gazebo reference="left_castor_dummy_link">
+		<material>Gazebo/DarkGrey</material>
+	</gazebo>
+	<gazebo reference="right_castor_dummy_link">
+		<material>Gazebo/DarkGrey</material>
 	</gazebo>
 <!-- ##################################################################### -->
@@ -210,25 +243,4 @@
 	<!-- DIFFERENTIAL DRIVE CONTROLLER -->
 	<gazebo>
-		<plugin name="differential_drive_controller_caster" filename="libgazebo_ros_diff_drive.so">
-			<legacyMode>false</legacyMode>
-			<rosDebugLevel>Debug</rosDebugLevel>
-			<publishWheelTF>true</publishWheelTF>
-			<robotNamespace>/</robotNamespace>
-			<publishTf>0</publishTf>
-			<broadcastTF>0</broadcastTF>
-			<alwaysOn>true</alwaysOn>
-			<publishWheelJointState>false</publishWheelJointState>
-			<updateRate>${rate_sensor}</updateRate>
-			<leftJoint>left_caster_joint</leftJoint>
-			<rightJoint>right_caster_joint</rightJoint>
-			<wheelSeparation>${base_y}</wheelSeparation>
-			<wheelDiameter>0.2</wheelDiameter>
-			<wheelTorque>30</wheelTorque>
-			<wheelAcceleration>1.8</wheelAcceleration>
-			<commandTopic>cmd_vel</commandTopic>
-			<robotBaseFrame>base_link</robotBaseFrame>
-			<odometryFrame>odom</odometryFrame>
-			<odometryTopic>odom</odometryTopic>
-		</plugin>
 		<plugin name="differential_drive_controller" filename="libgazebo_ros_diff_drive.so">
 			<alwaysOn>true</alwaysOn>
@@ -237,5 +249,5 @@
 			<robotNamespace>/</robotNamespace>
 			<publishWheelTF>false</publishWheelTF>
-			<publishWheelJointState>true</publishWheelJointState>
+			<publishWheelJointState>false</publishWheelJointState>
 			<publishTf>1</publishTf>
 			<updateRate>${rate_sensor}</updateRate>
@@ -247,29 +259,16 @@
 			<wheelAcceleration>1.8</wheelAcceleration>
 			<commandTopic>cmd_vel</commandTopic>
-			<robotBaseFrame>base_link</robotBaseFrame>
+			<robotBaseFrame>base_footprint</robotBaseFrame>
 			<odometryFrame>odom</odometryFrame>
 			<odometryTopic>odom</odometryTopic>
 			<odometrySource>world</odometrySource>
+			<publishOdom>true</publishOdom>
 		</plugin>
-		<plugin name="differential_drive_controller_top" filename="libgazebo_ros_diff_drive.so">
-			<legacyMode>false</legacyMode>
-			<rosDebugLevel>Debug</rosDebugLevel>
-			<publishWheelTF>true</publishWheelTF>
-			<robotNamespace>/</robotNamespace>
-			<publishTf>0</publishTf>
-			<broadcastTF>0</broadcastTF>
-			<alwaysOn>true</alwaysOn>
-			<publishWheelJointState>false</publishWheelJointState>
-			<updateRate>${rate_sensor}</updateRate>
-			<leftJoint>left_top_joint</leftJoint>
-			<rightJoint>right_top_joint</rightJoint>
-			<wheelSeparation>${base_y}</wheelSeparation>
-			<wheelDiameter>0.05</wheelDiameter>
-			<wheelTorque>30</wheelTorque>
-			<wheelAcceleration>1.8</wheelAcceleration>
-			<commandTopic>cmd_vel</commandTopic>
-			<robotBaseFrame>base_link</robotBaseFrame>
-			<odometryFrame>odom</odometryFrame>
-			<odometryTopic>odom</odometryTopic>
+	</gazebo>
+	<!-- ROS CONTROL -->
+	<gazebo>
+		<plugin name="gazebo_ros_control" filename="libgazebo_ros_control.so">
+		<legacyModeNS>false</legacyModeNS>
+		<robotNamespace>/</robotNamespace>
 		</plugin>
 	</gazebo>

File: wheelchair_description/urdf/wheelchair_property.xacro (robot description, xacro)
@@ -5,17 +5,24 @@
 	<xacro:property name="base_x" value="0.75" />
 	<xacro:property name="base_y" value="0.5" />
-	<xacro:property name="base_z" value="0.30" />
-	<xacro:property name="base_mass" value="5.0"/>
+	<xacro:property name="base_z" value="0.15" />
+	<xacro:property name="base_mass" value="100.0"/>
+	<xacro:property name="inertia_correcting_factor" value="20"/> <!-- aumenta l'inertia della base per ridurre il bug dello scivolamento, 1: no correction -->
 	<!-- Wheels -->
 	<xacro:property name="wheel_radius" value="0.2" />
 	<xacro:property name="wheel_height" value="0.1" />
-	<xacro:property name="wheel_mass" value="1" /> <!-- in kg-->
+	<xacro:property name="wheel_mass" value="5" />
 	<!-- Caster -->
-	<xacro:property name="caster_radius" value="0.1" />
-	<xacro:property name="caster_mass" value="0.5" /> <!-- in kg-->
-	<!-- Top -->
-	<xacro:property name="top_radius" value="0.025" />
-	<xacro:property name="top_height" value="0.2" />
-	<xacro:property name="top_mass" value="1" /> <!-- in kg-->
+	<xacro:property name="castor_mount_link_length" value="0.1" />
+	<xacro:property name="castor_mount_link_width" value="0.1" />
+	<xacro:property name="castor_mount_link_height" value="0.01" />
+	<xacro:property name="castor_mount_link_mass" value="0.25"/>
+	<xacro:property name="castor_dummy_link_length" value="0.02" />
+	<xacro:property name="castor_dummy_link_width" value="0.02" />
+	<xacro:property name="castor_dummy_link_height" value="0.02" />
+	<xacro:property name="castor_dummy_link_mass" value="0.25"/>
+	<xacro:property name="castor_wheel_length" value="0.1" />
+	<xacro:property name="castor_wheel_radius" value="0.095" />
+	<xacro:property name="castor_wheel_mass" value="2.5"/>
+	<xacro:property name="joint_friction" value="0.15" />
 	<!-- Material -->
 	<xacro:property name="d_grey" value="0.15"/>
@@ -27,5 +34,5 @@
 	<xacro:property name="imu_size" value="0.05"/>
 	<!-- Other -->
-	<xacro:property name="M_PI" value="3.14159265359" />
+	<xacro:property name="pi" value="3.14159265359" />
 	<xacro:property name="rate_sensor" value="50.0"/>
 </robot>

File: wheelchair_description/urdf/wheelchair_transmission.xacro (robot description, xacro)
@@ -2,9 +2,11 @@
 <robot xmlns:xacro="http://www.ros.org/wiki/xacro">
 	<!-- Wheels-->
-	<xacro:macro name="wheel_transmission" params="lr"> <!-- lr: left, right -->
-		<transmission name="${lr}_wheel_joint_trans">
+	<xacro:macro name="wheel_transmission" params="side">
+		<transmission name="${side}_wheel_joint_trans">
 			<type>transmission_interface/SimpleTransmission</type>
-			<joint name="${lr}_wheel_joint"/>
-			<actuator name="${lr}_wheel_joint_motor">
+			<joint name="${side}_wheel_joint">
+				<hardwareInterface>EffortJointInterface</hardwareInterface>
+			</joint>
+			<actuator name="${side}_wheel_joint_motor">
 				<hardwareInterface>EffortJointInterface</hardwareInterface>
 				<mechanicalReduction>1</mechanicalReduction>
@@ -12,31 +14,5 @@
 		</transmission>
     </xacro:macro>
-	<xacro:wheel_transmission lr="left" />
-	<xacro:wheel_transmission lr="right" />
-	<!-- Caster (non ci dovrebbe essere!!!) -->
-	<xacro:macro name="caster_transmission" params="lr"> <!-- lr: left, right -->
-		<transmission name="${lr}_caster_joint_trans">
-			<type>transmission_interface/SimpleTransmission</type>
-			<joint name="${lr}_caster_joint"/>
-			<actuator name="${lr}_caster_joint_motor">
-				<hardwareInterface>EffortJointInterface</hardwareInterface>
-				<mechanicalReduction>1</mechanicalReduction>
-			</actuator>
-		</transmission>
-    </xacro:macro>
-	<xacro:caster_transmission lr="left" />
-	<xacro:caster_transmission lr="right" />
-	<!-- Top (non ci dovrebbe essere!!!) -->
-	<xacro:macro name="top_transmission" params="lr"> <!-- lr: left, right -->
-		<transmission name="${lr}_top_joint_trans">
-			<type>transmission_interface/SimpleTransmission</type>
-			<joint name="${lr}_top_joint"/>
-			<actuator name="${lr}_top_joint_motor">
-				<hardwareInterface>EffortJointInterface</hardwareInterface>
-				<mechanicalReduction>1</mechanicalReduction>
-			</actuator>
-		</transmission>
-    </xacro:macro>
-	<xacro:top_transmission lr="left" />
-	<xacro:top_transmission lr="right" />
+	<xacro:wheel_transmission side="left" />
+	<xacro:wheel_transmission side="right" />
 </robot>

File: wheelchair_description/urdf/wheelchair_wheels.xacro (robot description, xacro)
@@ -1,13 +1,16 @@
 <?xml version="1.0"?>
 <robot xmlns:xacro="http://www.ros.org/wiki/xacro">
-	<!-- Wheels-->
 	<!-- Inertia matrix -->
 	<xacro:macro name="cylinder_inertia" params="m r h">
 		<inertia  ixx="${m*(3*r*r+h*h)/12}" ixy = "0" ixz = "0" iyy="${m*(3*r*r+h*h)/12}" iyz = "0" izz="${m*r*r/2}" />
 	</xacro:macro>
-	<xacro:macro name="wheel" params="lr parent translateX translateY translateZ flipY"> <!-- lr: left, right -->
-		<link name="${lr}_wheel">
+	<xacro:macro name="box_inertia" params="m w l h">
+		<inertia  ixx="${m*(w*w+h*h)/12}" ixy = "0" ixz = "0" iyy="${m*(l*l+h*h)/12}" iyz = "0" izz="${m*(l*l+h*h)/12}" />
+	</xacro:macro>
+	<!-- Wheels-->
+	<xacro:macro name="wheel" params="side translateX translateY translateZ">
+		<link name="${side}_wheel">
 			<visual>
-				<origin xyz="0 0 0" rpy="${flipY*M_PI/2} 0  0 " />
+				<origin xyz="0 0 0" rpy="${pi/2} 0 0"/>
 				<geometry>
 					<cylinder length="${wheel_height}" radius="${wheel_radius}" />
@@ -16,82 +19,124 @@
 			</visual>
 			<collision>
-				<origin xyz="0 0 0" rpy="${flipY*M_PI/2} 0 0" />
+				<origin xyz="0 0 0" rpy="${pi/2} 0 0"/>
 				<geometry><cylinder length="${wheel_height}" radius="${wheel_radius}" /></geometry>
 			</collision>
 			<inertial>
 				<mass value="${wheel_mass}" />
-				<origin xyz="0 0 0" />
-				<xacro:cylinder_inertia  m="${wheel_mass}" r="${wheel_radius}" h="${wheel_height}" />
+				<origin xyz="0 0 0" rpy="${pi/2} 0 0"/>
+				<xacro:cylinder_inertia  m="${wheel_mass}" r="${wheel_radius}" h="${wheel_height}"/>
 			</inertial>
 		</link>
-		<joint name="${lr}_wheel_joint" type="continuous">
-			<parent link="${parent}"/>
-			<child link="${lr}_wheel"/>
+		<joint name="${side}_wheel_joint" type="continuous">
+			<parent link="base_link"/>
+			<child link="${side}_wheel"/>
 			<origin xyz="${translateX} ${translateY} ${translateZ}" rpy="0 0 0" />
 			<axis xyz="0 1 0" />
 			<limit effort="100.0" lower="0.0" upper="0.0" velocity="100"/>
-			<joint_properties damping="0.0" friction="0.0"/>
+			<dynamics damping="0.0" friction="0.0"/>
 		</joint>
     </xacro:macro>
-	<xacro:wheel lr="right" parent="base_link" translateX="-0.15" translateY="-0.3" translateZ="-0.05" flipY="1" />
-	<xacro:wheel lr="left" parent="base_link" translateX="-0.15" translateY="0.3" translateZ="-0.05" flipY="1" />
+	<xacro:wheel side="right" translateX="-0.15" translateY="-0.3" translateZ="-0.125" />
+	<xacro:wheel side="left" translateX="-0.15" translateY="0.3" translateZ="-0.125" />
 	<!-- Caster -->
-	<xacro:macro name="caster" params="lr parent translateX translateY translateZ"> <!-- lr: left, right -->
-		<link name="${lr}_caster">
+	<xacro:macro name="caster" params="side X_mount Y_mount Z_mount X_dummy Y_dummy Z_dummy X_wheel Y_wheel Z_wheel">
+		<!-- caster mount link -->
+		<link name="${side}_castor_mount_link">
+			<collision>
+				<geometry>
+					<box size="${castor_mount_link_length} ${castor_mount_link_width} ${castor_mount_link_height}"/>
+				</geometry>
+				<origin xyz="0 0 0" rpy="0 0 0" />
+			</collision>
 			<visual>
-				<origin xyz="0 0 0" rpy="0 0  0 " />
 				<geometry>
-					<sphere radius="${caster_radius}" />
+					<box size="${castor_mount_link_length} ${castor_mount_link_width} ${castor_mount_link_height}"/>
 				</geometry>
+				<origin xyz="0 0 0" rpy="0 0 0" />
+				<material name="white"><color rgba="1 1 1 1"/></material>
+			</visual>
+			<inertial>
+				<origin xyz="0 0 0" rpy="0 0 0" />
+				<mass value="${castor_mount_link_mass}"/>
+				<xacro:box_inertia  m="${castor_mount_link_mass}"
+									w="${castor_mount_link_width}"
+									l="${castor_mount_link_length}"
+									h="${castor_mount_link_height}" />
+			</inertial>
+		</link>
+		<joint name="${side}_castor_mount_joint" type="fixed">
+			<parent link="base_link"/>
+			<child link="${side}_castor_mount_link"/>
+			<origin xyz="${X_mount} ${Y_mount} ${Z_mount}" />
+		</joint>
+		<!-- caster dummy link -->
+		<link name="${side}_castor_dummy_link">
+			<collision>
+				<geometry>
+					<box size="${castor_dummy_link_length} ${castor_dummy_link_width} ${castor_dummy_link_height}"/>
+				</geometry>
+				<origin xyz="0 0 0" rpy="0 0 0" />
+			</collision>
+			<visual>
+				<geometry>
+					<box size="${castor_dummy_link_length} ${castor_dummy_link_width} ${castor_dummy_link_height}"/>
+				</geometry>
+				<origin xyz="0 0 0" rpy="0 0 0" />
+				<material name="white"><color rgba="1 1 1 1"/></material>
+			</visual>
+			<inertial>
+				<origin xyz="0 0 0" rpy="0 0 0" />
+				<mass value="${castor_mount_link_mass}"/>
+				<xacro:box_inertia  m="${castor_dummy_link_mass}"
+									w="${castor_dummy_link_width}"
+									l="${castor_dummy_link_length}"
+									h="${castor_dummy_link_height}" />
+			</inertial>
+		</link>
+		<joint name="${side}_castor_dummy_joint" type="continuous">
+			<axis xyz="0 0 1"/>
+			<parent link="${side}_castor_mount_link"/>
+			<child link="${side}_castor_dummy_link"/>
+			<origin xyz="${X_dummy} ${Y_dummy} ${Z_dummy}" />
+			<dynamics friction="${joint_friction}"/>
+		</joint>
+		<!-- caster wheel -->
+		<link name="${side}_castor_wheel_link">
+			<collision>
+				<geometry>
+					<cylinder length="${castor_wheel_length}" radius="${castor_wheel_radius}"/>
+				</geometry>
+				<origin xyz="0 0 0" rpy="${pi/2} 0 0"/>
+			</collision>
+			<visual>
+				<geometry>
+					<cylinder length="${castor_wheel_length}" radius="${castor_wheel_radius}"/>
+				</geometry>
+				<origin xyz="0 0 0" rpy="${pi/2} 0 0"/>
 				<material name="grey"><color rgba="0.4 0.4 0.4 1"/></material>
 			</visual>
-			<collision>
-				<origin xyz="0 0 0" rpy="0 0 0" />
-				<geometry><sphere radius="${caster_radius}" /></geometry>
-			</collision>
 			<inertial>
-				<mass value="${caster_mass}"/>
-				<inertia ixx="0.0001" ixy="0.0" ixz="0.0" iyy="0.0001" iyz="0.0" izz="0.0001"/>
+				<origin xyz="0 0 0" rpy="${pi/2} 0 0"/>
+				<mass value="${castor_wheel_mass}"/>
+				<xacro:cylinder_inertia m="${castor_wheel_mass}"
+										r="${castor_wheel_radius}"
+										h="${castor_wheel_length}" />
 			</inertial>
 		</link>
-		<joint name="${lr}_caster_joint" type="continuous">
-			<parent link="${parent}"/>
-			<child link="${lr}_caster"/>
-			<origin xyz="${translateX} ${translateY} ${translateZ}" rpy="0 0 0" />
-			<axis xyz="0 1 0" />
+		<joint name="${side}_castor_wheel_joint" type="continuous">
+			<axis xyz="0 1 0"/>
+			<parent link="${side}_castor_dummy_link"/>
+			<child link="${side}_castor_wheel_link"/>
+			<origin xyz="${X_wheel} ${Y_wheel} ${Z_wheel}" />
+			<dynamics friction="${joint_friction}"/>
 		</joint>
     </xacro:macro>
-	<xacro:caster lr="left" parent="base_link" translateX="0.375" translateY="-0.275" translateZ="-0.15" />
-	<xacro:caster lr="right" parent="base_link" translateX="0.375" translateY="0.275" translateZ="-0.15" />
-	<!-- Top -->
-	<xacro:macro name="top" params="lr parent translateX translateY translateZ"> <!-- lr: left, right -->
-		<link name="${lr}_top">
-			<visual>
-				<origin xyz="0 0 0" rpy="0 0  0 " />
-				<geometry>
-					<cylinder length="${top_height}" radius="${top_radius}" />
-				</geometry>
-				<material name="white"><color rgba="1 1 1 1"/></material>
-			</visual>
-			<collision>
-				<origin xyz="0 0 0" rpy="0 0 0" />
-				<geometry><cylinder length="${top_height}" radius="${top_radius}" /></geometry>
-			</collision>
-			<inertial>
-				<mass value="${top_mass}" />
-				<origin xyz="0 0 0" />
-				<xacro:cylinder_inertia  m="${top_mass}" r="${top_radius}" h="${top_height}" />
-			</inertial>
-		</link>
-		<joint name="${lr}_top_joint" type="continuous">
-			<parent link="${parent}"/>
-			<child link="${lr}_top"/>
-			<origin xyz="${translateX} ${translateY} ${translateZ}" rpy="0 0 0" />
-			<axis xyz="0 0 1" />
-			<limit effort="100.0" lower="0.0" upper="0.0" velocity="100"/>
-			<joint_properties damping="0.0" friction="0.0"/>
-		</joint>
-    </xacro:macro>
-	<xacro:top lr="left" parent="base_link" translateX="0.375" translateY="-0.275" translateZ="0" />
-	<xacro:top lr="right" parent="base_link" translateX="0.375" translateY="0.275" translateZ="0" />
+	<xacro:caster side="left"
+				  X_mount="0.375" Y_mount="0.275" Z_mount="-0.09"
+				  X_dummy="0.0" Y_dummy="0.0" Z_dummy="-0.015"
+				  X_wheel="-0.05" Y_wheel="0.0" Z_wheel="-0.12" />
+	<xacro:caster side="right"
+				  X_mount="0.375" Y_mount="-0.275" Z_mount="-0.09"
+	  		      X_dummy="0.0" Y_dummy="0.0" Z_dummy="-0.015"
+				  X_wheel="-0.05" Y_wheel="0.0" Z_wheel="-0.12" />
 </robot>
