Commit message: Changelog:
-) Changed libgazebo_diff_drive with diff drive controller of ros_control;
-) Added robot_localization package to get odometry by fusing wheel odometry and imu.

File: wheelchair_description/urdf/wheelchair_gazebo.xacro (robot description, xacro)
@@ -101,5 +101,5 @@
 			<pose>${hokuyo_size/2} 0 0 0 0 0</pose>
 			<visualize>false</visualize>
-			<update_rate>${rate_sensor}</update_rate>
+			<update_rate>${hokuyo_rate}</update_rate>
 			<ray>
 				<scan>
@@ -124,76 +124,77 @@
 	</gazebo>
 	<!-- Imu -->
+	<!-- NB: nel plugin standard non sono supportati valori differenti di rumore per ang_vel, lin_acc, e orientamento. Va usato il plugin di hector per maggiori opzioni -->
 	<gazebo reference="imu_link">
 		<material>Gazebo/Orange</material>
 		<!-- <turnGravityOff>false</turnGravityOff> -->
 		<sensor type="imu" name="imu_sensor">
+		<!-- Sono supportati solo in sdf
 			<imu>
-				  <angular_velocity>
-				    <x>
-				      <noise type="gaussian">
-				        <mean>0.0</mean>
-				        <stddev>2e-4</stddev>
-				        <bias_mean>0.0000075</bias_mean>
-				        <bias_stddev>0.0000008</bias_stddev>
-				      </noise>
-				    </x>
-				    <y>
-				      <noise type="gaussian">
-				        <mean>0.0</mean>
-				        <stddev>2e-4</stddev>
-				        <bias_mean>0.0000075</bias_mean>
-				        <bias_stddev>0.0000008</bias_stddev>
-				      </noise>
-				    </y>
-				    <z>
-				      <noise type="gaussian">
-				        <mean>0.0</mean>
-				        <stddev>2e-4</stddev>
-				        <bias_mean>0.0000075</bias_mean>
-				        <bias_stddev>0.0000008</bias_stddev>
-				      </noise>
-				    </z>
-				  </angular_velocity>
-				  <linear_acceleration>
-				    <x>
-				      <noise type="gaussian">
-				        <mean>0.0</mean>
-				        <stddev>1.7e-2</stddev>
-				        <bias_mean>0.1</bias_mean>
-				        <bias_stddev>0.001</bias_stddev>
-				      </noise>
-				    </x>
-				    <y>
-				      <noise type="gaussian">
-				        <mean>0.0</mean>
-				        <stddev>1.7e-2</stddev>
-				        <bias_mean>0.1</bias_mean>
-				        <bias_stddev>0.001</bias_stddev>
-				      </noise>
-				    </y>
-				    <z>
-				      <noise type="gaussian">
-				        <mean>0.0</mean>
-				        <stddev>1.7e-2</stddev>
-				        <bias_mean>0.1</bias_mean>
-				        <bias_stddev>0.001</bias_stddev>
-				      </noise>
-				    </z>
-				  </linear_acceleration>
+				<angular_velocity>
+					<x>
+						<noise type="gaussian">
+						<mean>0.0</mean>
+						<stddev>2e-4</stddev>
+						<bias_mean>0.0000075</bias_mean>
+						<bias_stddev>0.0000008</bias_stddev>
+						</noise>
+					</x>
+					<y>
+						<noise type="gaussian">
+						<mean>0.0</mean>
+						<stddev>2e-4</stddev>
+						<bias_mean>0.0000075</bias_mean>
+						<bias_stddev>0.0000008</bias_stddev>
+						</noise>
+					</y>
+					<z>
+						<noise type="gaussian">
+						<mean>0.0</mean>
+						<stddev>2e-4</stddev>
+						<bias_mean>0.0000075</bias_mean>
+						<bias_stddev>0.0000008</bias_stddev>
+						</noise>
+					</z>
+				</angular_velocity>
+				<linear_acceleration>
+					<x>
+						<noise type="gaussian">
+						<mean>0.0</mean>
+						<stddev>1.7e-2</stddev>
+						<bias_mean>0.1</bias_mean>
+						<bias_stddev>0.001</bias_stddev>
+						</noise>
+					</x>
+					<y>
+						<noise type="gaussian">
+						<mean>0.0</mean>
+						<stddev>1.7e-2</stddev>
+						<bias_mean>0.1</bias_mean>
+						<bias_stddev>0.001</bias_stddev>
+						</noise>
+					</y>
+					<z>
+						<noise type="gaussian">
+						<mean>0.0</mean>
+						<stddev>1.7e-2</stddev>
+						<bias_mean>0.1</bias_mean>
+						<bias_stddev>0.001</bias_stddev>
+						</noise>
+					</z>
+				</linear_acceleration>
 			</imu>
+			-->
 			<pose>0 0 0 0 0 0</pose>
-			<update_rate>${rate_sensor}</update_rate>
+			<update_rate>${imu_rate}</update_rate>
     		<plugin name="gazebo_ros_imu_controller" filename="libgazebo_ros_imu_sensor.so">
-    	  		<topicName>/imu</topicName>
+				<alwaysOn>true</alwaysOn>
+				<topicName>/imu/data</topicName>
     	  		<frameName>imu_link</frameName>
-    	  		<alwaysOn>true</alwaysOn>
-    	  		<bodyName>base_link</bodyName>
-    	  		<gaussianNoise>0.5</gaussianNoise>
-    	  		<serviceName>imu/calibrate</serviceName>
+				<updateRateHZ>${imu_rate}</updateRateHZ>
+    	  		<bodyName>imu_link</bodyName>
+				<serviceName>imu/calibrate</serviceName>
+    	  		<gaussianNoise>0.0002</gaussianNoise>
     	  		<rpyOffset>0 0 0</rpyOffset>
-				<accelDrift>0.5 0.5 0.5</accelDrift>
-				<accelGaussianNoise>0.35 0.35 0.35</accelGaussianNoise>
-				<rateDrift>0.1 0.1 0.1</rateDrift>
-				<rateGaussianNoise>0.05 0.05 0.05</rateGaussianNoise>
+				<initialOrientationAsReference>false</initialOrientationAsReference>
     		</plugin>
     	</sensor>
@@ -203,5 +204,5 @@
 		<material>Gazebo/Red</material>
 		<sensor type="camera" name="camera_sensor">
-		  <update_rate>${rate_sensor}</update_rate>
+		  <update_rate>${camera_rate}</update_rate>
 		  <camera>
 			<horizontal_fov>1.047197551</horizontal_fov> <!--60 gradi-->
@@ -241,6 +242,27 @@
   </gazebo>
 <!-- ##################################################################### -->
+	<!-- ROS CONTROL -->
+	<gazebo>
+		<plugin name="gazebo_ros_control" filename="libgazebo_ros_control.so">
+		<legacyModeNS>false</legacyModeNS>
+		<robotNamespace>/</robotNamespace>
+		</plugin>
+	</gazebo>
+	<!-- GROUND TRUTH ODOMETRY -->
+	<gazebo>
+		<plugin name="p3d_base_controller" filename="libgazebo_ros_p3d.so">
+			<alwaysOn>true</alwaysOn>
+			<updateRate>50.0</updateRate>
+			<bodyName>base_footprint</bodyName>
+			<topicName>ground_truth_odom</topicName>
+			<gaussianNoise>0.0</gaussianNoise>
+			<frameName>map</frameName>
+			<xyzOffsets>0 0 0</xyzOffsets>
+			<rpyOffsets>0 0 0</rpyOffsets>
+		</plugin>
+	</gazebo>
 	<!-- DIFFERENTIAL DRIVE CONTROLLER -->
-	<gazebo>
+	<!-- Sostituito dal diff drive controller di ros control -->
+	<!-- <gazebo>
 		<plugin name="differential_drive_controller" filename="libgazebo_ros_diff_drive.so">
 			<alwaysOn>true</alwaysOn>
@@ -250,9 +272,10 @@
 			<publishWheelTF>false</publishWheelTF>
 			<publishWheelJointState>false</publishWheelJointState>
-			<publishTf>1</publishTf>
-			<updateRate>${rate_sensor}</updateRate>
+			<publishTf>${with_odom}</publishTf>
+			<publishOdom>true</publishOdom>
+			<updateRate>${encoder_rate}</updateRate>
 			<leftJoint>left_wheel_joint</leftJoint>
 			<rightJoint>right_wheel_joint</rightJoint>
-			<wheelSeparation>${base_y}</wheelSeparation>
+			<wheelSeparation>${base_y + wheel_height}</wheelSeparation>
 			<wheelDiameter>${2*wheel_radius}</wheelDiameter>
 			<wheelTorque>30</wheelTorque>
@@ -263,13 +286,5 @@
 			<odometryTopic>odom</odometryTopic>
 			<odometrySource>world</odometrySource>
-			<publishOdom>true</publishOdom>
 		</plugin>
-	</gazebo>
-	<!-- ROS CONTROL -->
-	<gazebo>
-		<plugin name="gazebo_ros_control" filename="libgazebo_ros_control.so">
-		<legacyModeNS>false</legacyModeNS>
-		<robotNamespace>/</robotNamespace>
-		</plugin>
-	</gazebo>
+	</gazebo> -->
 </robot>

File: wheelchair_description/urdf/wheelchair_property.xacro (robot description, xacro)
@@ -1,4 +1,13 @@
 <?xml version="1.0"?>
 <robot xmlns:xacro="http://www.ros.org/wiki/xacro">
+	<!-- ARG FROM LAUNCH FILE -->
+	<!-- <xacro:arg name="localization" default="" /> <~~! True: odom from custom algorithm. False: odom from gazebo diff drive.~~>
+	<xacro:if value="$(arg localization)">
+		<xacro:property name="with_odom" value="false" /> <~~! Odom from custom algorithm. ~~>
+	</xacro:if>
+	<xacro:unless value="$(arg localization)">
+		<xacro:property name="with_odom" value="true" /> <~~! Odom from gazebo diff drive. ~~>
+	</xacro:unless>
+	 -->
 	<!-- PROPERTY LIST -->
 	<!-- Base -->
@@ -29,10 +38,14 @@
 	<!-- Camera -->
 	<xacro:property name="camera_size" value="0.05" />
+	<xacro:property name="camera_rate" value="50.0"/>
 	<!-- Hokuyo -->
 	<xacro:property name="hokuyo_size" value="0.05"/>
+	<xacro:property name="hokuyo_rate" value="50.0"/>
 	<!-- Imu -->
 	<xacro:property name="imu_size" value="0.05"/>
+	<xacro:property name="imu_rate" value="100"/>
+	<!-- Encoder -->
+	<xacro:property name="encoder_rate" value="50.0"/>
 	<!-- Other -->
-	<xacro:property name="pi" value="3.14159265359" />
-	<xacro:property name="rate_sensor" value="50.0"/>
+	<xacro:property name="PI" value="3.14159265359" />
 </robot>

File: wheelchair_description/urdf/wheelchair_transmission.xacro (robot description, xacro)
@@ -6,8 +6,8 @@
 			<type>transmission_interface/SimpleTransmission</type>
 			<joint name="${side}_wheel_joint">
-				<hardwareInterface>EffortJointInterface</hardwareInterface>
+				<hardwareInterface>hardware_interface/VelocityJointInterface</hardwareInterface>
 			</joint>
 			<actuator name="${side}_wheel_joint_motor">
-				<hardwareInterface>EffortJointInterface</hardwareInterface>
+				<hardwareInterface>hardware_interface/VelocityJointInterface</hardwareInterface>
 				<mechanicalReduction>1</mechanicalReduction>
 			</actuator>

File: wheelchair_description/urdf/wheelchair_wheels.xacro (robot description, xacro)
@@ -12,5 +12,5 @@
 		<link name="${side}_wheel">
 			<visual>
-				<origin xyz="0 0 0" rpy="${pi/2} 0 0"/>
+				<origin xyz="0 0 0" rpy="${PI/2} 0 0"/>
 				<geometry>
 					<cylinder length="${wheel_height}" radius="${wheel_radius}" />
@@ -19,10 +19,10 @@
 			</visual>
 			<collision>
-				<origin xyz="0 0 0" rpy="${pi/2} 0 0"/>
+				<origin xyz="0 0 0" rpy="${PI/2} 0 0"/>
 				<geometry><cylinder length="${wheel_height}" radius="${wheel_radius}" /></geometry>
 			</collision>
 			<inertial>
 				<mass value="${wheel_mass}" />
-				<origin xyz="0 0 0" rpy="${pi/2} 0 0"/>
+				<origin xyz="0 0 0" rpy="${PI/2} 0 0"/>
 				<xacro:cylinder_inertia  m="${wheel_mass}" r="${wheel_radius}" h="${wheel_height}"/>
 			</inertial>
@@ -107,5 +107,5 @@
 					<cylinder length="${castor_wheel_length}" radius="${castor_wheel_radius}"/>
 				</geometry>
-				<origin xyz="0 0 0" rpy="${pi/2} 0 0"/>
+				<origin xyz="0 0 0" rpy="${PI/2} 0 0"/>
 			</collision>
 			<visual>
@@ -113,9 +113,9 @@
 					<cylinder length="${castor_wheel_length}" radius="${castor_wheel_radius}"/>
 				</geometry>
-				<origin xyz="0 0 0" rpy="${pi/2} 0 0"/>
+				<origin xyz="0 0 0" rpy="${PI/2} 0 0"/>
 				<material name="grey"><color rgba="0.4 0.4 0.4 1"/></material>
 			</visual>
 			<inertial>
-				<origin xyz="0 0 0" rpy="${pi/2} 0 0"/>
+				<origin xyz="0 0 0" rpy="${PI/2} 0 0"/>
 				<mass value="${castor_wheel_mass}"/>
 				<xacro:cylinder_inertia m="${castor_wheel_mass}"

Commit message: Changelog
-) Fix for rotational drift with ekf
-) Tuned parameters for diff-corrected model of AMCL
-) Added a node to broadcast, if necessary, the TF odom->base_footprint from ground truth odometry values
-) Added the costmap of small_office world

File: wheelchair_description/urdf/wheelchair_gazebo.xacro (robot description, xacro)
@@ -194,5 +194,5 @@
     	  		<bodyName>imu_link</bodyName>
 				<serviceName>imu/calibrate</serviceName>
-    	  		<gaussianNoise>0.0002</gaussianNoise>
+    	  		<gaussianNoise>0.001</gaussianNoise>
     	  		<rpyOffset>0 0 0</rpyOffset>
 				<initialOrientationAsReference>false</initialOrientationAsReference>
@@ -255,5 +255,5 @@
 			<updateRate>50.0</updateRate>
 			<bodyName>base_footprint</bodyName>
-			<topicName>ground_truth_odom</topicName>
+			<topicName>/odometry/ground_truth_odom</topicName>
 			<gaussianNoise>0.0</gaussianNoise>
 			<frameName>map</frameName>

File: wheelchair_description/urdf/wheelchair_property.xacro (robot description, xacro)
@@ -44,8 +44,6 @@
 	<!-- Imu -->
 	<xacro:property name="imu_size" value="0.05"/>
-	<xacro:property name="imu_rate" value="100"/>
+	<xacro:property name="imu_rate" value="300"/>
 	<!-- Encoder -->
 	<xacro:property name="encoder_rate" value="50.0"/>
-	<!-- Other -->
-	<xacro:property name="PI" value="3.14159265359" />
 </robot>

File: wheelchair_description/urdf/wheelchair_sensors.xacro (robot description, xacro)
@@ -31,5 +31,5 @@
 	</link>
 	<joint name="imu_joint" type="fixed">
-    	<origin xyz="${-base_x/2 + imu_size} 0 ${base_z/2+imu_size/2}" rpy="0 0 0"/>
+    	<origin xyz="${-base_x/2 + imu_size} 0 ${base_z/2+imu_size/2}" rpy="0 0 ${0}"/>
     	<parent link="base_link"/>
     	<child link="imu_link"/>

File: wheelchair_description/urdf/wheelchair_wheels.xacro (robot description, xacro)
@@ -12,5 +12,5 @@
 		<link name="${side}_wheel">
 			<visual>
-				<origin xyz="0 0 0" rpy="${PI/2} 0 0"/>
+				<origin xyz="0 0 0" rpy="${pi/2} 0 0"/>
 				<geometry>
 					<cylinder length="${wheel_height}" radius="${wheel_radius}" />
@@ -19,10 +19,10 @@
 			</visual>
 			<collision>
-				<origin xyz="0 0 0" rpy="${PI/2} 0 0"/>
+				<origin xyz="0 0 0" rpy="${pi/2} 0 0"/>
 				<geometry><cylinder length="${wheel_height}" radius="${wheel_radius}" /></geometry>
 			</collision>
 			<inertial>
 				<mass value="${wheel_mass}" />
-				<origin xyz="0 0 0" rpy="${PI/2} 0 0"/>
+				<origin xyz="0 0 0" rpy="${pi/2} 0 0"/>
 				<xacro:cylinder_inertia  m="${wheel_mass}" r="${wheel_radius}" h="${wheel_height}"/>
 			</inertial>
@@ -107,5 +107,5 @@
 					<cylinder length="${castor_wheel_length}" radius="${castor_wheel_radius}"/>
 				</geometry>
-				<origin xyz="0 0 0" rpy="${PI/2} 0 0"/>
+				<origin xyz="0 0 0" rpy="${pi/2} 0 0"/>
 			</collision>
 			<visual>
@@ -113,9 +113,9 @@
 					<cylinder length="${castor_wheel_length}" radius="${castor_wheel_radius}"/>
 				</geometry>
-				<origin xyz="0 0 0" rpy="${PI/2} 0 0"/>
+				<origin xyz="0 0 0" rpy="${pi/2} 0 0"/>
 				<material name="grey"><color rgba="0.4 0.4 0.4 1"/></material>
 			</visual>
 			<inertial>
-				<origin xyz="0 0 0" rpy="${PI/2} 0 0"/>
+				<origin xyz="0 0 0" rpy="${pi/2} 0 0"/>
 				<mass value="${castor_wheel_mass}"/>
 				<xacro:cylinder_inertia m="${castor_wheel_mass}"
