Commit message: Added ros_control diff-effort control loop. Added a sample simulated hardware interface for ros_control controllers.

File: wheelchair_description/urdf/wheelchair_gazebo_old.xacro (robot description, xacro)
@@ -247,5 +247,4 @@
 		<legacyModeNS>false</legacyModeNS>
 		<robotNamespace>/</robotNamespace>
-		<robotSimType>${robot_interface}</robotSimType>
 		</plugin>
 	</gazebo>

File: wheelchair_description/urdf/wheelchair_property_old.xacro (robot description, xacro)
@@ -2,7 +2,12 @@
 <robot xmlns:xacro="http://www.ros.org/wiki/xacro">
 	<!-- ARG FROM LAUNCH FILE -->
-	<xacro:arg name="use_sample_interface" default="false" />
-	<xacro:arg name="use_effort" default="false" />
-	<!-- ******************************************************************************************************************************** -->
+	<!-- <xacro:arg name="localization" default="" /> <~~! True: odom from custom algorithm. False: odom from gazebo diff drive.~~>
+	<xacro:if value="$(arg localization)">
+		<xacro:property name="with_odom" value="false" /> <~~! Odom from custom algorithm. ~~>
+	</xacro:if>
+	<xacro:unless value="$(arg localization)">
+		<xacro:property name="with_odom" value="true" /> <~~! Odom from gazebo diff drive. ~~>
+	</xacro:unless>
+	 -->
 	<!-- PROPERTY LIST -->
 	<!-- Base -->
@@ -42,16 +47,3 @@
 	<!-- Encoder -->
 	<xacro:property name="encoder_rate" value="50.0"/>
-	<!-- Other -->
-	<xacro:if value="$(arg use_sample_interface)">
-		 <xacro:property name="robot_interface" value="wheelchair_gazebo_interface/WheelchairHardwareSim" />
-	</xacro:if>
-	<xacro:unless value="$(arg use_sample_interface)">
-		 <xacro:property name="robot_interface" value="gazebo_ros_control/DefaultRobotHWSim" /> <!--<~~! . ~~> -->
-	</xacro:unless>
-	<xacro:if value="$(arg use_effort)">
-		 <xacro:property name="hw_interface" value="hardware_interface/EffortJointInterface" />
-	</xacro:if>
-	<xacro:unless value="$(arg use_effort)">
-		 <xacro:property name="hw_interface" value="hardware_interface/VelocityJointInterface" />
-	</xacro:unless>
 </robot>

File: wheelchair_description/urdf/wheelchair_transmission_old.xacro (robot description, xacro)
@@ -6,8 +6,8 @@
 			<type>transmission_interface/SimpleTransmission</type>
 			<joint name="${side}_wheel_joint">
-				<hardwareInterface>${hw_interface}</hardwareInterface>
+				<hardwareInterface>hardware_interface/VelocityJointInterface</hardwareInterface>
 			</joint>
 			<actuator name="${side}_wheel_joint_motor">
-				<hardwareInterface>${hw_interface}</hardwareInterface>
+				<hardwareInterface>hardware_interface/VelocityJointInterface</hardwareInterface>
 				<mechanicalReduction>1</mechanicalReduction>
 			</actuator>
